Commit message: diff_car: fit sth. for vlp lidar

File: src/diff_car/urdf/camera.xacro (robot description, xacro)
@@ -4,5 +4,5 @@
   <xacro:property name="camera_width" value="0.025" />
   <xacro:property name="camera_height" value="0.025" />
-  <xacro:property name="camera_x" value="0.03" />
+  <xacro:property name="camera_x" value="0.02" />
   <xacro:property name="camera_y" value="0.0" />
   <xacro:property name="camera_z" value="${laser_length / 2 + camera_height / 2}" />

File: src/diff_car/urdf/car_vlp.xacro (robot description, xacro)
@@ -4,10 +4,10 @@
   <xacro:include filename="base.xacro" />
   <xacro:include filename="laser.xacro" />
+  <xacro:include filename="laser_driver.xacro" />
   <xacro:include filename="imu.xacro" />
+  <xacro:include filename="imu_driver.xacro" />
   <xacro:include filename="camera.xacro" />
-  <xacro:include filename="move.xacro" />
-  <xacro:include filename="laser_driver.xacro" />
-  <xacro:include filename="imu_driver.xacro" />
   <xacro:include filename="camera_driver.xacro" />
   <xacro:include filename="imu_pose_gt.xacro" />
+  <xacro:include filename="move.xacro" />
 </robot>
